Commit message: [WIP] 椅子の土台まで出来た

File: human_model_gazebo/urdf/human.xacro (robot description, xacro)
@@ -7,15 +7,16 @@
   <xacro:property name="deg_to_rad" value="0.01745329251994329577"/>
   <!-- Constants for robot dimensions -->
-  <xacro:property name="length" value="0.5" />
-  <xacro:property name="width" value="0.3" />
+  <xacro:property name="length" value="0.4" />
+  <xacro:property name="width" value="0.4" />
   <xacro:property name="wheel_radius" value="0.11" /> <!-- Link 1 -->
   <xacro:property name="thickness" value="0.086" /> <!-- Link 2 -->
   <xacro:property name="axel_offset" value="0.05" /> <!-- Space btw top of beam and the each joint -->
   <xacro:property name="steer_offset" value="0.02" /> <!-- Link 1 -->
+  <xacro:property name="steer_height" value="0.4" />
   <!-- Links: inertial,visual,collision -->
   <link name="base_link">
     <inertial>
       <!-- origin is relative -->
-      <origin xyz="0 0 0.4" rpy="0 0 0"/>
+      <origin xyz="0 0 0.2" rpy="0 0 0"/>
       <mass value="5"/>
       <inertia ixx="5" ixy="0" ixz="0" iyy="5" iyz="0" izz="5"/>
@@ -23,5 +24,5 @@
     <visual>
       <geometry>
-        <box size="${length} ${width} 0.1"/>
+        <box size="${length} ${width} 0.05"/>
       </geometry>
     </visual>
@@ -54,11 +55,26 @@
   <!-- Wheels -->
   <front_wheel name="front_right" parent="base" radius="${wheel_radius}" thickness="${thickness}"
-      length="${length}" width="${width}" axel_offset="${axel_offset}" right_left="1" steer_height="${wheel_radius+steer_offset}">
-    <origin xyz="${length/2-axel_offset} ${width/2+axel_offset} 0" rpy="${-90 * deg_to_rad} 0 0"/>
+      length="${length}" width="${width}" axel_offset="${axel_offset}" right_left="1" steer_height="${steer_height}">
   </front_wheel>
   <front_wheel name="front_left" parent="base" radius="${wheel_radius}" thickness="${thickness}"
+      length="${length}" width="${width}" axel_offset="${axel_offset}" right_left="-1" steer_height="${steer_height}">
+  </front_wheel>
+  <rear_wheel name="rear_right" parent="base" radius="${wheel_radius}" thickness="${thickness}"
+      length="${length}" width="${width}" axel_offset="${axel_offset}" right_left="1" steer_height="${steer_height}">
+  </rear_wheel>
+  <rear_wheel name="rear_left" parent="base" radius="${wheel_radius}" thickness="${thickness}"
+      length="${length}" width="${width}" axel_offset="${axel_offset}" right_left="-1" steer_height="${steer_height}">
+  </rear_wheel>
+  <!--
+  <front_wheel name="rear_right" parent="base" radius="${wheel_radius}" thickness="${thickness}"
+      length="${length}" width="${width}" axel_offset="${axel_offset}" right_left="1" steer_height="${wheel_radius+steer_offset}">
+    <origin xyz="${-(length/2-axel_offset)} ${width/2+axel_offset} 0" rpy="${-90 * deg_to_rad} 0 0"/>
+  </front_wheel>
+  <front_wheel name="rear_left" parent="base" radius="${wheel_radius}" thickness="${thickness}"
       length="${length}" width="${width}" axel_offset="${axel_offset}" right_left="-1" steer_height="${wheel_radius+steer_offset}">
-    <origin xyz="${length/2-axel_offset} ${-width/2-axel_offset} 0" rpy="${-90 * deg_to_rad} 0 0"/>
+    <origin xyz="${-(length/2-axel_offset)} ${-width/2-axel_offset} 0" rpy="${-90 * deg_to_rad} 0 0"/>
   </front_wheel>
+  -->
+  <!--
   <rear_wheel name="rear_right" parent="base" radius="${wheel_radius}" thickness="${thickness}">
     <origin xyz="${-length/2+axel_offset} ${width/2+axel_offset} 0" rpy="${-90 * deg_to_rad} 0 0"/>
@@ -67,7 +83,8 @@
     <origin xyz="${-length/2+axel_offset} ${-width/2-axel_offset} 0" rpy="${-90 * deg_to_rad} 0 0"/>
   </rear_wheel>
+  -->
   <!-- Colour -->
   <gazebo reference="base_link">
-    <material>Gazebo/Green</material>
+    <material>Gazebo/WoodFloor</material>
   </gazebo>
   <gazebo reference="base_footprint">

File: human_model_gazebo/urdf/wheel.xacro (robot description, xacro)
@@ -1,25 +1,24 @@
 <?xml version="1.0"?>
 <robot xmlns:xacro="http://www.ros.org/wiki/xacro">
-  <xacro:property name="steer_radius" value="0.05" /> <!-- Link 1 -->
-  <xacro:property name="steer_thickness" value="0.02" /> <!-- Link 1 -->
+  <xacro:property name="steer_radius" value="0.04" /> <!-- Link 1 -->
   <xacro:property name="steer_effort"   value="10.0"/>
   <xacro:property name="steer_velocity" value="5.0"/>
-  <macro name="front_wheel" params="name parent radius thickness length width axel_offset right_left steer_height *origin">
+  <macro name="front_wheel" params="name parent radius thickness length width axel_offset right_left steer_height ">
     <link name="${name}_steer_link">
       <inertial>
-        <origin xyz="0 0 0" rpy="0 0 0"/>
+        <origin xyz="0 0 0.4" rpy="0 0 0"/>
         <mass value="1"/>
         <inertia ixx="0.2" ixy="0" ixz="0" iyy="0.2" iyz="0" izz="0.2"/>
       </inertial>
       <visual>
-        <origin xyz="0 0 0" rpy="0 0 0"/>
+        <origin xyz="0 0 0.2" rpy="0 0 0"/>
         <geometry>
-          <cylinder radius="${steer_radius}" length="${steer_thickness}"/>
+          <cylinder radius="${steer_radius}" length="${steer_height}"/>
         </geometry>
       </visual>
       <collision>
-        <origin xyz="0 0 0" rpy="0 0 0"/>
+        <origin xyz="0 0 0.2" rpy="0 0 0"/>
         <geometry>
-          <cylinder radius="${steer_radius}" length="${steer_thickness}"/>
+          <cylinder radius="${steer_radius}" length="${steer_height}"/>
         </geometry>
       </collision>
@@ -28,5 +27,5 @@
       <parent link="${parent}_link"/>
       <child link="${name}_steer_link"/>
-      <origin xyz="${length/2-axel_offset} ${right_left*(width/2+axel_offset)} ${steer_height}" rpy="0 0 0"/>
+      <origin xyz="${length/2-axel_offset} ${right_left*(width/2-axel_offset)} ${-steer_height}" rpy="0 0 0"/>
       <!--insert_block name="origin"/-->
       <axis xyz="0 0 1"/>
@@ -35,42 +34,44 @@
              velocity="${steer_velocity}"/>
      </joint>
-    <link name="${name}_wheel_link">
+    <gazebo reference="${name}_steer_link">
+      <material>Gazebo/WoodFloor</material>
+    </gazebo>
+    <gazebo reference="${name}_wheel_link">
+      <material>Gazebo/WoodFloor</material>
+    </gazebo>
+  </macro>
+  <macro name="rear_wheel" params="name parent radius thickness length width axel_offset right_left steer_height ">
+    <link name="${name}_steer_link">
       <inertial>
-        <origin xyz="0 0 0" rpy="0 0 0"/>
+        <origin xyz="0 0 0.4" rpy="0 0 0"/>
         <mass value="1"/>
         <inertia ixx="0.2" ixy="0" ixz="0" iyy="0.2" iyz="0" izz="0.2"/>
       </inertial>
       <visual>
-        <origin xyz="0 0 0" rpy="0 0 0"/>
+        <origin xyz="0 0 0.2" rpy="0 0 0"/>
         <geometry>
-          <cylinder radius="${wheel_radius}" length="${thickness}"/>
+          <cylinder radius="${steer_radius}" length="${steer_height}"/>
         </geometry>
       </visual>
       <collision>
-        <origin xyz="0 0 0" rpy="0 0 0"/>
+        <origin xyz="0 0 0.2" rpy="0 0 0"/>
         <geometry>
-          <cylinder radius="${wheel_radius}" length="${thickness}"/>
+          <cylinder radius="${steer_radius}" length="${steer_height}"/>
         </geometry>
       </collision>
     </link>
-    <joint name="${name}_wheel_joint" type="continuous">
-      <parent link="${name}_steer_link"/>
-      <child link="${name}_wheel_link"/>
-      <origin xyz="0 0 ${-steer_height}" rpy="${-90 * deg_to_rad} 0 0"/>
+    <joint name="${name}_steer_joint" type="revolute">
+      <parent link="${parent}_link"/>
+      <child link="${name}_steer_link"/>
+      <origin xyz="${-(length/2-axel_offset)} ${right_left*(width/2-axel_offset)} ${-steer_height}" rpy="0 0 0"/>
+      <!--insert_block name="origin"/-->
       <axis xyz="0 0 1"/>
-    </joint>
-    <!-- Transmission is important to link the joints and the controller -->
-    <transmission name="${name}_steer_joint_trans" type="SimpleTransmission">
-      <actuator name="${name}_steer_joint_motor"/>
-      <joint name="${name}_steer_joint"/>
-      <mechanicalReduction>1</mechanicalReduction>
-      <motorTorqueConstant>1</motorTorqueConstant>
-    </transmission>
-    <transmission name="${name}_wheel_joint_trans" type="SimpleTransmission">
-      <actuator name="${name}_wheel_joint_motor"/>
-      <joint name="${name}_wheel_joint"/>
-      <mechanicalReduction>1</mechanicalReduction>
-      <motorTorqueConstant>1</motorTorqueConstant>
-    </transmission>
+      <limit effort="${steer_effort}"
+             lower="${-180.0 * deg_to_rad}" upper="${180.0 * deg_to_rad}"
+             velocity="${steer_velocity}"/>
+     </joint>
+    <gazebo reference="${name}_steer_link">
+      <material>Gazebo/WoodFloor</material>
+    </gazebo>
     <gazebo reference="${name}_steer_link">
       <material>Gazebo/Blue</material>
@@ -80,5 +81,5 @@
     </gazebo>
   </macro>
-  <macro name="rear_wheel" params="name parent radius thickness *origin">
+  <!--macro name="rear_wheel" params="name parent radius thickness *origin">
     <link name="${name}_wheel_link">
       <inertial>
@@ -106,5 +107,4 @@
       <axis xyz="0 0 1"/>
     </joint>
-    <!-- Transmission is important to link the joints and the controller -->
     <transmission name="${name}_wheel_joint_trans" type="SimpleTransmission">
       <actuator name="${name}_wheel_joint_motor"/>
@@ -116,4 +116,4 @@
       <material>Gazebo/Red</material>
     </gazebo>
-  </macro>
+  </macro-->
 </robot>

Commit message: [WIP] 椅子の背もたれまで出来た．

File: human_model_gazebo/urdf/human.xacro (robot description, xacro)
@@ -24,5 +24,5 @@
     <visual>
       <geometry>
-        <box size="${length} ${width} 0.05"/>
+        <box size="${length} ${width} 0.04"/>
       </geometry>
     </visual>
@@ -52,4 +52,30 @@
     <child link="base_link"/>
     <parent link="base_footprint"/>
+  </joint>
+  <!-- Links: inertial,visual,collision -->
+  <link name="back_link">
+    <inertial>
+      <!-- origin is relative -->
+      <origin xyz="0 0 0" rpy="0 0 0"/>
+      <mass value="5"/>
+      <inertia ixx="5" ixy="0" ixz="0" iyy="5" iyz="0" izz="5"/>
+    </inertial>
+    <visual>
+      <geometry>
+        <box size="${length} ${width} 0.04"/>
+      </geometry>
+    </visual>
+    <collision>
+      <!-- origin is relative -->
+      <origin xyz="0 0 0"/>
+      <geometry>
+        <box size="${length} ${width} 0.1"/>
+      </geometry>
+    </collision>
+  </link>
+  <joint name="base_back_joint" type="fixed">
+      <origin xyz="${-length/2.0+0.02} 0 ${length/2.0}" rpy="0 ${-90 * deg_to_rad} 0"/>
+    <child link="back_link"/>
+    <parent link="base_link"/>
   </joint>
   <!-- Wheels -->
@@ -88,4 +114,7 @@
     <material>Gazebo/WoodFloor</material>
   </gazebo>
+  <gazebo reference="back_link">
+    <material>Gazebo/WoodFloor</material>
+  </gazebo>
   <gazebo reference="base_footprint">
     <material>Gazebo/Purple</material>

File: human_model_gazebo/urdf/wheel.xacro (robot description, xacro)
@@ -1,5 +1,5 @@
 <?xml version="1.0"?>
 <robot xmlns:xacro="http://www.ros.org/wiki/xacro">
-  <xacro:property name="steer_radius" value="0.04" /> <!-- Link 1 -->
+  <xacro:property name="steer_radius" value="0.03" /> <!-- Link 1 -->
   <xacro:property name="steer_effort"   value="10.0"/>
   <xacro:property name="steer_velocity" value="5.0"/>
@@ -74,10 +74,4 @@
       <material>Gazebo/WoodFloor</material>
     </gazebo>
-    <gazebo reference="${name}_steer_link">
-      <material>Gazebo/Blue</material>
-    </gazebo>
-    <gazebo reference="${name}_wheel_link">
-      <material>Gazebo/Red</material>
-    </gazebo>
   </macro>
   <!--macro name="rear_wheel" params="name parent radius thickness *origin">

Commit message: [WIP] 横のボードまで出来た．

File: human_model_gazebo/urdf/human.xacro (robot description, xacro)
@@ -14,4 +14,6 @@
   <xacro:property name="steer_offset" value="0.02" /> <!-- Link 1 -->
   <xacro:property name="steer_height" value="0.4" />
+  <xacro:property name="board_length" value="0.8" />
+  <xacro:property name="board_width" value="0.3" />
   <!-- Links: inertial,visual,collision -->
   <link name="base_link">
@@ -31,5 +33,5 @@
       <origin xyz="0 0 0"/>
       <geometry>
-        <box size="${length} ${width} 0.1"/>
+        <box size="${length} ${width} 0.04"/>
       </geometry>
     </collision>
@@ -70,11 +72,63 @@
       <origin xyz="0 0 0"/>
       <geometry>
-        <box size="${length} ${width} 0.1"/>
+        <box size="${length} ${width} 0.04"/>
       </geometry>
     </collision>
   </link>
   <joint name="base_back_joint" type="fixed">
-      <origin xyz="${-length/2.0+0.02} 0 ${length/2.0}" rpy="0 ${-90 * deg_to_rad} 0"/>
+      <origin xyz="${-length/2.0 + 0.02} 0 ${length/2.0}" rpy="0 ${-90 * deg_to_rad} 0"/>
     <child link="back_link"/>
+    <parent link="base_link"/>
+  </joint>
+  <!-- Links: inertial,visual,collision -->
+  <link name="panelfront_link">
+    <inertial>
+      <!-- origin is relative -->
+      <origin xyz="0 0 0" rpy="0 0 0"/>
+      <mass value="5"/>
+      <inertia ixx="5" ixy="0" ixz="0" iyy="5" iyz="0" izz="5"/>
+    </inertial>
+    <visual>
+      <geometry>
+        <box size="${board_length} ${board_width} 0.02"/>
+      </geometry>
+    </visual>
+    <collision>
+      <!-- origin is relative -->
+      <origin xyz="0 0 0"/>
+      <geometry>
+        <box size="${board_length} ${board_width} 0.02"/>
+      </geometry>
+    </collision>
+  </link>
+  <joint name="base_panelfront_joint" type="fixed">
+      <origin xyz="0.08 0.45 -0.005" rpy="0 ${80 * deg_to_rad} 0"/>
+    <child link="panelfront_link"/>
+    <parent link="base_link"/>
+  </joint>
+  <!-- Links: inertial,visual,collision -->
+  <link name="panelback_link">
+    <inertial>
+      <!-- origin is relative -->
+      <origin xyz="0 0 0" rpy="0 0 0"/>
+      <mass value="5"/>
+      <inertia ixx="5" ixy="0" ixz="0" iyy="5" iyz="0" izz="5"/>
+    </inertial>
+    <visual>
+      <geometry>
+        <box size="${board_length} ${board_width} 0.02"/>
+      </geometry>
+    </visual>
+    <collision>
+      <!-- origin is relative -->
+      <origin xyz="0 0 0"/>
+      <geometry>
+        <box size="${board_length} ${board_width} 0.02"/>
+      </geometry>
+    </collision>
+  </link>
+  <joint name="base_panelback_joint" type="fixed">
+     <origin xyz="-0.08 0.45 -0.005" rpy="0 ${-80 * deg_to_rad} 0"/>
+    <child link="panelback_link"/>
     <parent link="base_link"/>
   </joint>
@@ -117,4 +171,10 @@
     <material>Gazebo/WoodFloor</material>
   </gazebo>
+  <gazebo reference="panelfront_link">
+    <material>Gazebo/Yellow</material>
+  </gazebo>
+  <gazebo reference="panelback_link">
+    <material>Gazebo/Yellow</material>
+  </gazebo>
   <gazebo reference="base_footprint">
     <material>Gazebo/Purple</material>

Commit message: [WIP] 下半身まで出来た．

File: human_model_gazebo/urdf/human.xacro (robot description, xacro)
@@ -164,4 +164,231 @@
   </rear_wheel>
   -->
+  <!-- Links: inertial,visual,collision -->
+  <link name="body_link">
+    <inertial>
+      <!-- origin is relative -->
+      <origin xyz="0 0 0" rpy="0 0 0"/>
+      <mass value="5"/>
+      <inertia ixx="5" ixy="0" ixz="0" iyy="5" iyz="0" izz="5"/>
+    </inertial>
+    <visual>
+      <geometry>
+        <box size="${length} 0.25 0.1"/>
+      </geometry>
+    </visual>
+    <collision>
+      <!-- origin is relative -->
+      <origin xyz="0 0 0"/>
+      <geometry>
+        <box size="${length} 0.25 0.1"/>
+      </geometry>
+    </collision>
+  </link>
+  <joint name="base_body_joint" type="fixed">
+      <origin xyz="-0.0 0 ${length/2.0}" rpy="0 ${-90 * deg_to_rad} 0"/>
+    <child link="body_link"/>
+    <parent link="base_link"/>
+  </joint>
+  <link name="bodyright_link">
+    <inertial>
+      <!-- origin is relative -->
+      <origin xyz="0 0 0" rpy="0 0 0"/>
+      <mass value="5"/>
+      <inertia ixx="5" ixy="0" ixz="0" iyy="5" iyz="0" izz="5"/>
+    </inertial>
+    <visual>
+      <geometry>
+        <cylinder radius="0.05" length="${length}"/>
+      </geometry>
+    </visual>
+    <collision>
+      <!-- origin is relative -->
+      <origin xyz="0 0 0"/>
+      <geometry>
+        <cylinder radius="0.05" length="${length}"/>
+      </geometry>
+    </collision>
+  </link>
+  <joint name="body_bodyright_joint" type="fixed">
+      <origin xyz="0.0 -0.125 0" rpy="0 ${-90 * deg_to_rad} 0"/>
+    <child link="bodyright_link"/>
+    <parent link="body_link"/>
+  </joint>
+  <!-- left leg -->
+  <link name="bodyleft_link">
+    <inertial>
+      <!-- origin is relative -->
+      <origin xyz="0 0 0" rpy="0 0 0"/>
+      <mass value="5"/>
+      <inertia ixx="5" ixy="0" ixz="0" iyy="5" iyz="0" izz="5"/>
+    </inertial>
+    <visual>
+      <geometry>
+        <cylinder radius="0.05" length="${length}"/>
+      </geometry>
+    </visual>
+    <collision>
+      <!-- origin is relative -->
+      <origin xyz="0 0 0"/>
+      <geometry>
+        <cylinder radius="0.05" length="${length}"/>
+      </geometry>
+    </collision>
+  </link>
+  <joint name="body_bodyleft_joint" type="fixed">
+      <origin xyz="0.0 0.125 0" rpy="0 ${-90 * deg_to_rad} 0"/>
+    <child link="bodyleft_link"/>
+    <parent link="body_link"/>
+  </joint>
+  <link name="legright1_link">
+    <inertial>
+      <!-- origin is relative -->
+      <origin xyz="0 0 0" rpy="0 0 0"/>
+      <mass value="5"/>
+      <inertia ixx="5" ixy="0" ixz="0" iyy="5" iyz="0" izz="5"/>
+    </inertial>
+    <visual>
+      <geometry>
+        <cylinder radius="0.05" length="0.25"/>
+      </geometry>
+    </visual>
+    <collision>
+      <!-- origin is relative -->
+      <origin xyz="0 0 0"/>
+      <geometry>
+       <cylinder radius="0.05" length="0.25"/>
+      </geometry>
+    </collision>
+  </link>
+  <joint name="bodyright_legright1_joint" type="fixed">
+      <origin xyz="-0.2 0 0.125" rpy="0 ${-90 * deg_to_rad} 0"/>
+    <child link="legright1_link"/>
+    <parent link="bodyright_link"/>
+  </joint>
+  <link name="legleft1_link">
+    <inertial>
+      <!-- origin is relative -->
+      <origin xyz="0 0 0" rpy="0 0 0"/>
+      <mass value="5"/>
+      <inertia ixx="5" ixy="0" ixz="0" iyy="5" iyz="0" izz="5"/>
+    </inertial>
+    <visual>
+      <geometry>
+        <cylinder radius="0.05" length="0.25"/>
+      </geometry>
+    </visual>
+    <collision>
+      <!-- origin is relative -->
+      <origin xyz="0 0 0"/>
+      <geometry>
+        <cylinder radius="0.05" length="0.25"/>
+      </geometry>
+    </collision>
+  </link>
+  <joint name="bodyleft_legleft1__joint" type="fixed">
+      <origin xyz="-0.2 0 0.125" rpy="0 ${-90 * deg_to_rad} 0"/>
+    <child link="legleft1_link"/>
+    <parent link="bodyleft_link"/>
+  </joint>
+  <link name="legright2_link">
+    <inertial>
+      <!-- origin is relative -->
+      <origin xyz="0 0 0" rpy="0 0 0"/>
+      <mass value="5"/>
+      <inertia ixx="5" ixy="0" ixz="0" iyy="5" iyz="0" izz="5"/>
+    </inertial>
+    <visual>
+      <geometry>
+        <sphere radius="0.05"/>
+      </geometry>
+    </visual>
+    <collision>
+      <!-- origin is relative -->
+      <origin xyz="0 0 0"/>
+      <geometry>
+        <sphere radius="0.05"/>
+      </geometry>
+    </collision>
+  </link>
+  <joint name="legright1_legright2__joint" type="fixed">
+      <origin xyz="0 0 0.125" rpy="0 0 0"/>
+    <child link="legright2_link"/>
+    <parent link="legright1_link"/>
+  </joint>
+  <link name="legleft2_link">
+    <inertial>
+      <!-- origin is relative -->
+      <origin xyz="0 0 0" rpy="0 0 0"/>
+      <mass value="5"/>
+      <inertia ixx="5" ixy="0" ixz="0" iyy="5" iyz="0" izz="5"/>
+    </inertial>
+    <visual>
+      <geometry>
+        <sphere radius="0.05"/>
+      </geometry>
+    </visual>
+    <collision>
+      <!-- origin is relative -->
+      <origin xyz="0 0 0"/>
+      <geometry>
+        <sphere radius="0.05"/>
+      </geometry>
+    </collision>
+  </link>
+  <joint name="legleft1_legleft2__joint" type="fixed">
+      <origin xyz="0 0 0.125" rpy="0 0 0"/>
+    <child link="legleft2_link"/>
+    <parent link="legleft1_link"/>
+  </joint>
+  <link name="legleft3_link">
+    <inertial>
+      <!-- origin is relative -->
+      <origin xyz="0 0 0" rpy="0 0 0"/>
+      <mass value="5"/>
+      <inertia ixx="5" ixy="0" ixz="0" iyy="5" iyz="0" izz="5"/>
+    </inertial>
+    <visual>
+      <geometry>
+        <cylinder radius="0.05" length="0.45"/>
+      </geometry>
+    </visual>
+    <collision>
+      <!-- origin is relative -->
+      <origin xyz="0 0 0"/>
+      <geometry>
+        <cylinder radius="0.05" length="0.45"/>
+      </geometry>
+    </collision>
+  </link>
+  <joint name="legleft2_legleft3__joint" type="fixed">
+      <origin xyz="0.225 0 0" rpy="0 ${-90 * deg_to_rad} 0"/>
+    <child link="legleft3_link"/>
+    <parent link="legleft2_link"/>
+  </joint>
+  <link name="legright3_link">
+    <inertial>
+      <!-- origin is relative -->
+      <origin xyz="0 0 0" rpy="0 0 0"/>
+      <mass value="5"/>
+      <inertia ixx="5" ixy="0" ixz="0" iyy="5" iyz="0" izz="5"/>
+    </inertial>
+    <visual>
+      <geometry>
+        <cylinder radius="0.05" length="0.45"/>
+      </geometry>
+    </visual>
+    <collision>
+      <!-- origin is relative -->
+      <origin xyz="0 0 0"/>
+      <geometry>
+        <cylinder radius="0.05" length="0.45"/>
+      </geometry>
+    </collision>
+  </link>
+  <joint name="legright2_legright3__joint" type="fixed">
+      <origin xyz="0.225 0 0" rpy="0 ${-90 * deg_to_rad} 0"/>
+    <child link="legright3_link"/>
+    <parent link="legright2_link"/>
+  </joint>
   <!-- Colour -->
   <gazebo reference="base_link">
@@ -180,3 +407,6 @@
     <material>Gazebo/Purple</material>
   </gazebo>
+  <gazebo reference="body_link">
+    <material>Gazebo/White</material>
+  </gazebo>
 </robot>
