Commit message: [WIP] 下半身足も出来た．

File: human_model_gazebo/urdf/human.xacro (robot description, xacro)
@@ -7,4 +7,5 @@
   <xacro:property name="deg_to_rad" value="0.01745329251994329577"/>
   <!-- Constants for robot dimensions -->
+  <xacro:property name="human_back_length" value="0.5" />
   <xacro:property name="length" value="0.4" />
   <xacro:property name="width" value="0.4" />
@@ -65,5 +66,5 @@
     <visual>
       <geometry>
-        <box size="${length} ${width} 0.04"/>
+        <box size="${human_back_length} ${width} 0.04"/>
       </geometry>
     </visual>
@@ -174,17 +175,17 @@
     <visual>
       <geometry>
-        <box size="${length} 0.25 0.1"/>
-      </geometry>
-    </visual>
-    <collision>
-      <!-- origin is relative -->
-      <origin xyz="0 0 0"/>
-      <geometry>
-        <box size="${length} 0.25 0.1"/>
+        <box size="${human_back_length} 0.25 0.1"/>
+      </geometry>
+    </visual>
+    <collision>
+      <!-- origin is relative -->
+      <origin xyz="0 0 0"/>
+      <geometry>
+        <box size="${human_back_length} 0.25 0.1"/>
       </geometry>
     </collision>
   </link>
   <joint name="base_body_joint" type="fixed">
-      <origin xyz="-0.0 0 ${length/2.0}" rpy="0 ${-90 * deg_to_rad} 0"/>
+      <origin xyz="-0.0 0 ${human_back_length/2.0}" rpy="0 ${-90 * deg_to_rad} 0"/>
     <child link="body_link"/>
     <parent link="base_link"/>
@@ -199,12 +200,12 @@
     <visual>
       <geometry>
-        <cylinder radius="0.05" length="${length}"/>
-      </geometry>
-    </visual>
-    <collision>
-      <!-- origin is relative -->
-      <origin xyz="0 0 0"/>
-      <geometry>
-        <cylinder radius="0.05" length="${length}"/>
+        <cylinder radius="0.05" length="${human_back_length}"/>
+      </geometry>
+    </visual>
+    <collision>
+      <!-- origin is relative -->
+      <origin xyz="0 0 0"/>
+      <geometry>
+        <cylinder radius="0.05" length="${human_back_length}"/>
       </geometry>
     </collision>
@@ -225,12 +226,12 @@
     <visual>
       <geometry>
-        <cylinder radius="0.05" length="${length}"/>
-      </geometry>
-    </visual>
-    <collision>
-      <!-- origin is relative -->
-      <origin xyz="0 0 0"/>
-      <geometry>
-        <cylinder radius="0.05" length="${length}"/>
+        <cylinder radius="0.05" length="${human_back_length}"/>
+      </geometry>
+    </visual>
+    <collision>
+      <!-- origin is relative -->
+      <origin xyz="0 0 0"/>
+      <geometry>
+        <cylinder radius="0.05" length="${human_back_length}"/>
       </geometry>
     </collision>
@@ -262,5 +263,5 @@
   </link>
   <joint name="bodyright_legright1_joint" type="fixed">
-      <origin xyz="-0.2 0 0.125" rpy="0 ${-90 * deg_to_rad} 0"/>
+      <origin xyz="-0.2 0 ${human_back_length/2-0.075}" rpy="0 ${-90 * deg_to_rad} 0"/>
     <child link="legright1_link"/>
     <parent link="bodyright_link"/>
@@ -287,5 +288,5 @@
   </link>
   <joint name="bodyleft_legleft1__joint" type="fixed">
-      <origin xyz="-0.2 0 0.125" rpy="0 ${-90 * deg_to_rad} 0"/>
+      <origin xyz="-0.2 0 ${human_back_length/2-0.075}" rpy="0 ${-90 * deg_to_rad} 0"/>
     <child link="legleft1_link"/>
     <parent link="bodyleft_link"/>
@@ -391,4 +392,55 @@
     <parent link="legright2_link"/>
   </joint>
+  <link name="footleft_link">
+    <inertial>
+      <!-- origin is relative -->
+      <origin xyz="0 0 0" rpy="0 0 0"/>
+      <mass value="5"/>
+      <inertia ixx="5" ixy="0" ixz="0" iyy="5" iyz="0" izz="5"/>
+    </inertial>
+    <visual>
+      <geometry>
+        <box size="0.2 0.1 0.08"/>
+      </geometry>
+    </visual>
+    <collision>
+      <!-- origin is relative -->
+      <origin xyz="0 0 0"/>
+      <geometry>
+        <box size="0.2 0.1 0.05"/>
+      </geometry>
+    </collision>
+  </link>
+  <joint name="legleft3_footleft_joint" type="fixed">
+      <origin xyz="0.05 0 -${0.45*0.5}" rpy="0 0 0"/>
+    <child link="footleft_link"/>
+    <parent link="legleft3_link"/>
+  </joint>
+  <link name="footright_link">
+    <inertial>
+      <!-- origin is relative -->
+      <origin xyz="0 0 0" rpy="0 0 0"/>
+      <mass value="5"/>
+      <inertia ixx="5" ixy="0" ixz="0" iyy="5" iyz="0" izz="5"/>
+    </inertial>
+    <visual>
+      <geometry>
+        <box size="0.2 0.1 0.08"/>
+      </geometry>
+    </visual>
+    <collision>
+      <!-- origin is relative -->
+      <origin xyz="0 0 0"/>
+      <geometry>
+        <box size="0.2 0.1 0.05"/>
+      </geometry>
+    </collision>
+  </link>
+  <joint name="legrihgt3_footrihgt_joint" type="fixed">
+      <origin xyz="0.05 0 -${0.45*0.5}" rpy="0 0 0"/>
+    <child link="footright_link"/>
+    <parent link="legright3_link"/>
+  </joint>
+  <!-- Arm -->
   <!-- Colour -->
   <gazebo reference="base_link">

Commit message: [WIP] 肩までできた

File: human_model_gazebo/urdf/human.xacro (robot description, xacro)
@@ -39,9 +39,9 @@
   </link>
   <link name="base_footprint">
-    <visual>
+    <!--visual>
       <geometry>
         <sphere radius="0.01"/>
       </geometry>
-    </visual>
+    </visual-->
     <collision>
       <origin xyz="0 0 0"/>
@@ -442,5 +442,81 @@
     <parent link="legright3_link"/>
   </joint>
+  <!-- Chest -->
+  <link name="chest_link">
+    <inertial>
+      <!-- origin is relative -->
+      <origin xyz="0 0 0" rpy="0 0 0"/>
+      <mass value="5"/>
+      <inertia ixx="5" ixy="0" ixz="0" iyy="5" iyz="0" izz="5"/>
+    </inertial>
+    <visual>
+      <geometry>
+        <cylinder radius="0.05" length="0.25"/>
+      </geometry>
+    </visual>
+    <collision>
+      <!-- origin is relative -->
+      <origin xyz="0 0 0"/>
+      <geometry>
+        <cylinder radius="0.05" length="0.25"/>
+      </geometry>
+    </collision>
+  </link>
+  <joint name="body_chest_joint" type="fixed">
+      <origin xyz="0.25 0 0" rpy="${-90 * deg_to_rad} 0 0"/>
+    <child link="chest_link"/>
+    <parent link="body_link"/>
+  </joint>
   <!-- Arm -->
+  <link name="shoulderleft_link">
+    <inertial>
+      <!-- origin is relative -->
+      <origin xyz="0 0 0" rpy="0 0 0"/>
+      <mass value="5"/>
+      <inertia ixx="5" ixy="0" ixz="0" iyy="5" iyz="0" izz="5"/>
+    </inertial>
+    <visual>
+      <geometry>
+        <sphere radius="0.05"/>
+      </geometry>
+    </visual>
+    <collision>
+      <!-- origin is relative -->
+      <origin xyz="0 0 0"/>
+      <geometry>
+        <sphere radius="0.05"/>
+      </geometry>
+    </collision>
+  </link>
+  <joint name="bodyleft_shoulderleft_joint" type="fixed">
+      <origin xyz="0 0 -0.25" rpy="0 0 0"/>
+    <child link="shoulderleft_link"/>
+    <parent link="bodyleft_link"/>
+  </joint>
+  <link name="shoulderright_link">
+    <inertial>
+      <!-- origin is relative -->
+      <origin xyz="0 0 0" rpy="0 0 0"/>
+      <mass value="5"/>
+      <inertia ixx="5" ixy="0" ixz="0" iyy="5" iyz="0" izz="5"/>
+    </inertial>
+    <visual>
+      <geometry>
+        <sphere radius="0.05"/>
+      </geometry>
+    </visual>
+    <collision>
+      <!-- origin is relative -->
+      <origin xyz="0 0 0"/>
+      <geometry>
+        <sphere radius="0.05"/>
+      </geometry>
+    </collision>
+  </link>
+  <joint name="bodyright_shoulderright_joint" type="fixed">
+      <origin xyz="0 0 -0.25" rpy="0 0 0"/>
+    <child link="shoulderright_link"/>
+    <parent link="bodyright_link"/>
+  </joint>
   <!-- Colour -->
   <gazebo reference="base_link">

Commit message: [add] human model完成

File: human_model_gazebo/urdf/human.xacro (robot description, xacro)
@@ -242,8 +242,8 @@
     <parent link="body_link"/>
   </joint>
-  <link name="legright1_link">
-    <inertial>
-      <!-- origin is relative -->
-      <origin xyz="0 0 0" rpy="0 0 0"/>
+0  <link name="legright1_link">
+    <inertial>
+      <!-- origin is relative -->
+0gin xyz="0 0 0" rpy="0 0 0"/>
       <mass value="5"/>
       <inertia ixx="5" ixy="0" ixz="0" iyy="5" iyz="0" izz="5"/>
@@ -287,5 +287,5 @@
     </collision>
   </link>
-  <joint name="bodyleft_legleft1__joint" type="fixed">
+  <joint name="bodyleft_legleft1_joint" type="fixed">
       <origin xyz="-0.2 0 ${human_back_length/2-0.075}" rpy="0 ${-90 * deg_to_rad} 0"/>
     <child link="legleft1_link"/>
@@ -312,5 +312,5 @@
     </collision>
   </link>
-  <joint name="legright1_legright2__joint" type="fixed">
+  <joint name="legright1_legright2_joint" type="fixed">
       <origin xyz="0 0 0.125" rpy="0 0 0"/>
     <child link="legright2_link"/>
@@ -337,5 +337,5 @@
     </collision>
   </link>
-  <joint name="legleft1_legleft2__joint" type="fixed">
+  <joint name="legleft1_legleft2_joint" type="fixed">
       <origin xyz="0 0 0.125" rpy="0 0 0"/>
     <child link="legleft2_link"/>
@@ -362,5 +362,5 @@
     </collision>
   </link>
-  <joint name="legleft2_legleft3__joint" type="fixed">
+  <joint name="legleft2_legleft3_joint" type="fixed">
       <origin xyz="0.225 0 0" rpy="0 ${-90 * deg_to_rad} 0"/>
     <child link="legleft3_link"/>
@@ -387,5 +387,5 @@
     </collision>
   </link>
-  <joint name="legright2_legright3__joint" type="fixed">
+  <joint name="legright2_legright3_joint" type="fixed">
       <origin xyz="0.225 0 0" rpy="0 ${-90 * deg_to_rad} 0"/>
     <child link="legright3_link"/>
@@ -468,4 +468,30 @@
     <parent link="body_link"/>
   </joint>
+  <!-- Head -->
+  <link name="head_link">
+    <inertial>
+      <!-- origin is relative -->
+      <origin xyz="0 0 0" rpy="0 0 0"/>
+      <mass value="5"/>
+      <inertia ixx="5" ixy="0" ixz="0" iyy="5" iyz="0" izz="5"/>
+    </inertial>
+    <visual>
+      <geometry>
+        <sphere radius="0.125"/>
+      </geometry>
+    </visual>
+    <collision>
+      <!-- origin is relative -->
+      <origin xyz="0 0 0"/>
+      <geometry>
+        <sphere radius="0.125"/>
+      </geometry>
+    </collision>
+  </link>
+  <joint name="chest_head_joint" type="fixed">
+      <origin xyz="0.15 0 0" rpy="0 0 0"/>
+    <child link="head_link"/>
+    <parent link="chest_link"/>
+  </joint>
   <!-- Arm -->
   <link name="shoulderleft_link">
@@ -518,4 +544,204 @@
     <child link="shoulderright_link"/>
     <parent link="bodyright_link"/>
+  </joint>
+  <link name="armright1_link">
+    <inertial>
+      <!-- origin is relative -->
+      <origin xyz="0 0 0" rpy="0 0 0"/>
+      <mass value="5"/>
+      <inertia ixx="5" ixy="0" ixz="0" iyy="5" iyz="0" izz="5"/>
+    </inertial>
+    <visual>
+      <geometry>
+        <cylinder radius="0.05" length="0.25"/>
+      </geometry>
+    </visual>
+    <collision>
+      <!-- origin is relative -->
+      <origin xyz="0 0 0"/>
+      <geometry>
+        <cylinder radius="0.05" length="0.25"/>
+      </geometry>
+    </collision>
+  </link>
+  <joint name="shoulderright_armright1_joint" type="fixed">
+      <origin xyz="-0.065 0 0.11" rpy="0 ${-30 * deg_to_rad} 0"/>
+    <child link="armright1_link"/>
+    <parent link="shoulderright_link"/>
+  </joint>
+  <link name="armleft1_link">
+    <inertial>
+      <!-- origin is relative -->
+      <origin xyz="0 0 0" rpy="0 0 0"/>
+      <mass value="5"/>
+      <inertia ixx="5" ixy="0" ixz="0" iyy="5" iyz="0" izz="5"/>
+    </inertial>
+    <visual>
+      <geometry>
+        <cylinder radius="0.05" length="0.25"/>
+      </geometry>
+    </visual>
+    <collision>
+      <!-- origin is relative -->
+      <origin xyz="0 0 0"/>
+      <geometry>
+        <cylinder radius="0.05" length="0.25"/>
+      </geometry>
+    </collision>
+  </link>
+  <joint name="shoulderleft_armleft1_joint" type="fixed">
+      <origin xyz="-0.065 0 0.11" rpy="0 ${-30 * deg_to_rad} 0"/>
+    <child link="armleft1_link"/>
+    <parent link="shoulderleft_link"/>
+  </joint>
+  <link name="armright2_link">
+    <inertial>
+      <!-- origin is relative -->
+      <origin xyz="0 0 0" rpy="0 0 0"/>
+      <mass value="5"/>
+      <inertia ixx="5" ixy="0" ixz="0" iyy="5" iyz="0" izz="5"/>
+    </inertial>
+    <visual>
+      <geometry>
+        <sphere radius="0.05"/>
+      </geometry>
+    </visual>
+    <collision>
+      <!-- origin is relative -->
+      <origin xyz="0 0 0"/>
+      <geometry>
+        <sphere radius="0.05"/>
+      </geometry>
+    </collision>
+  </link>
+  <joint name="armright1_armright2_joint" type="fixed">
+      <origin xyz="0 0 0.125" rpy="0 0 0"/>
+    <child link="armright2_link"/>
+    <parent link="armright1_link"/>
+  </joint>
+  <link name="armleft2_link">
+    <inertial>
+      <!-- origin is relative -->
+      <origin xyz="0 0 0" rpy="0 0 0"/>
+      <mass value="5"/>
+      <inertia ixx="5" ixy="0" ixz="0" iyy="5" iyz="0" izz="5"/>
+    </inertial>
+    <visual>
+      <geometry>
+        <sphere radius="0.05"/>
+      </geometry>
+    </visual>
+    <collision>
+      <!-- origin is relative -->
+      <origin xyz="0 0 0"/>
+      <geometry>
+        <sphere radius="0.05"/>
+      </geometry>
+    </collision>
+  </link>
+  <joint name="armleft1_armleft2_joint" type="fixed">
+      <origin xyz="0 0 0.125" rpy="0 0 0"/>
+    <child link="armleft2_link"/>
+    <parent link="armleft1_link"/>
+  </joint>
+  <link name="armleft3_link">
+    <inertial>
+      <!-- origin is relative -->
+      <origin xyz="0 0 0" rpy="0 0 0"/>
+      <mass value="5"/>
+      <inertia ixx="5" ixy="0" ixz="0" iyy="5" iyz="0" izz="5"/>
+    </inertial>
+    <visual>
+      <geometry>
+        <cylinder radius="0.05" length="0.2"/>
+      </geometry>
+    </visual>
+    <collision>
+      <!-- origin is relative -->
+      <origin xyz="0 0 0"/>
+      <geometry>
+        <cylinder radius="0.05" length="0.2"/>
+      </geometry>
+    </collision>
+  </link>
+  <joint name="armleft2_armleft3_joint" type="fixed">
+      <origin xyz="-0.065 0 0.11" rpy="0 ${-30 * deg_to_rad} 0"/>
+    <child link="armleft3_link"/>
+    <parent link="armleft2_link"/>
+  </joint>
+  <link name="armright3_link">
+    <inertial>
+      <!-- origin is relative -->
+      <origin xyz="0 0 0" rpy="0 0 0"/>
+      <mass value="5"/>
+      <inertia ixx="5" ixy="0" ixz="0" iyy="5" iyz="0" izz="5"/>
+    </inertial>
+    <visual>
+      <geometry>
+        <cylinder radius="0.05" length="0.2"/>
+      </geometry>
+    </visual>
+    <collision>
+      <!-- origin is relative -->
+      <origin xyz="0 0 0"/>
+      <geometry>
+        <cylinder radius="0.05" length="0.2"/>
+      </geometry>
+    </collision>
+  </link>
+  <joint name="armright2_armright3_joint" type="fixed">
+      <origin xyz="-0.065 0 0.11" rpy="0 ${-30 * deg_to_rad} 0"/>
+    <child link="armright3_link"/>
+    <parent link="armright2_link"/>
+  </joint>
+  <link name="handright_link">
+    <inertial>
+      <!-- origin is relative -->
+      <origin xyz="0 0 0" rpy="0 0 0"/>
+      <mass value="5"/>
+      <inertia ixx="5" ixy="0" ixz="0" iyy="5" iyz="0" izz="5"/>
+    </inertial>
+    <visual>
+      <geometry>
+        <sphere radius="0.065"/>
+      </geometry>
+    </visual>
+    <collision>
+      <!-- origin is relative -->
+      <origin xyz="0 0 0"/>
+      <geometry>
+        <sphere radius="0.065"/>
+      </geometry>
+    </collision>
+  </link>
+  <joint name="armrighht3_handright_joint" type="fixed">
+      <origin xyz="0 0 ${0.2*0.5}" rpy="0 0 0"/>
+    <child link="handright_link"/>
+    <parent link="armright3_link"/>
+  </joint>
+  <link name="handleft_link">
+    <inertial>
+      <!-- origin is relative -->
+      <origin xyz="0 0 0" rpy="0 0 0"/>
+      <mass value="5"/>
+      <inertia ixx="5" ixy="0" ixz="0" iyy="5" iyz="0" izz="5"/>
+    </inertial>
+    <visual>
+      <geometry>
+        <sphere radius="0.065"/>
+      </geometry>
+    </visual>
+    <collision>
+      <!-- origin is relative -->
+      <origin xyz="0 0 0"/>
+      <geometry>
+        <sphere radius="0.065"/>
+      </geometry>
+    </collision>
+  </link>
+  <joint name="armleft3_handleft_joint" type="fixed">
+      <origin xyz="0 0 ${0.2*0.5}" rpy="0 0 0"/>
+    <child link="handleft_link"/>
+    <parent link="armleft3_link"/>
   </joint>
   <!-- Colour -->
